File: Ontvanger/Ontvanger.kicad_sch (KiCad schematic)
At the start: 19 parts, among them IC1 STM32WB30CEU5A, IC2 QAM-RX10-433, J1 Conn_01x04_Male, U1 BAT-HLD-001

Commit message: filss added
Parts:
- removed Q?: Q_PMOS_DSG, symbol Device:Q_PMOS_DSG
- added Q1: AO3401A, Package_TO_SOT_SMD:SOT-23, symbol Transistor_FET:AO3401A
- IC2: footprint QAMRX10433 -> KiCad libs:QAMRX10433
- R1, R2, R3, R4: renamed from R?; footprint Resistor_SMD:R_4020_10251Metric -> Resistor_SMD:R_0201_0603Metric
- U1: footprint BATHLD001 -> KiCad libs:BATHLD001
- gave numbers to parts that had none: 10
Connections:
- net GND: no longer C2.1, U1.3, U2.3 (VBAT)
- net at C3.1, L1.1, R3.1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: now also Q1.3 (D)
- net at C1.1, D1.2 (A), J2.1 (VBUS)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: now also Q1.1 (G)
- new net: C2.1, Q1.2 (S), U1.3, U2.3 (VBAT)
